File: keyboard-pcb.kicad_sch (KiCad schematic)
At the start: 24 parts, among them J1 USB_B_Micro, SW1 SW_Push, U1 ATmega32U4-A, Y1 16Mhz

Commit message: changes2
Parts:
- J1: footprint (none) -> random-keyboard-parts:Molex-0548190589
- SW1: footprint random-keyboard-parts:Molex-0548190589 -> random-keyboard-parts:SKQG-1155865
Changed lines of the file:
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@@
     (property "Reference" "J1" (id 0) (at 121.92 50.8 0))
     (property "Value" "USB_B_Micro" (id 1) (at 121.92 53.34 0))
-    (property "Footprint" "" (id 2) (at 125.73 64.77 0)
+    (property "Footprint" "random-keyboard-parts:Molex-0548190589" (id 2) (at 125.73 64.77 0)
       (effects (font (size 1.27 1.27)) hide)
     )
@@
     (property "Reference" "SW1" (id 0) (at 57.15 50.8 0))
     (property "Value" "SW_Push" (id 1) (at 57.15 53.34 0))
-    (property "Footprint" "random-keyboard-parts:Molex-0548190589" (id 2) (at 57.15 53.34 0)
+    (property "Footprint" "random-keyboard-parts:SKQG-1155865" (id 2) (at 57.15 53.34 0)
       (effects (font (size 1.27 1.27)) hide)
     )
@@
     )
     (path "/286123f0-4f5c-443b-958e-bff37057547e"
-      (reference "J1") (unit 1) (value "USB_B_Micro") (footprint "")
+      (reference "J1") (unit 1) (value "USB_B_Micro") (footprint "random-keyboard-parts:Molex-0548190589")
     )
     (path "/152fc720-f34f-4984-812b-795bdc9a95ce"
@@
     )
     (path "/85096f46-9dbf-4764-9bad-58dbd71db34c"
-      (reference "SW1") (unit 1) (value "SW_Push") (footprint "random-keyboard-parts:Molex-0548190589")
+      (reference "SW1") (unit 1) (value "SW_Push") (footprint "random-keyboard-parts:SKQG-1155865")
     )
     (path "/3e7be21d-6b73-43ce-85e9-9d2bc1b07b9b"
